Commit message: Minnor changes

File: go2_description/urdf/go2.xacro.urdf (robot description, URDF)
Before this commit: robot go2, 33 links, 32 joints
Links:
- removed link base_footprint
- removed link map
- removed link odom
- added link torso, mass 6.921; collision box size=0.3762 0.0935 0.114; visual mesh filename=package://go2_description/dae/base.dae
- added link world
- link base_link: mass 6.921 -> None; geometry 
Joints:
- removed joint base_footprint_joint
- removed joint map_joint
- removed joint odom_joint
- added joint fixed: type fixed, parent world, child base_link, origin xyz=0 0 1
- added joint joint_fixed_: type fixed, parent base_link, child torso, origin xyz=0 0 0.5
- joint FL_hip_joint: parent base_link -> torso
- joint FR_hip_joint: parent base_link -> torso
- joint Head_upper_joint: parent base_link -> torso
- joint RL_hip_joint: parent base_link -> torso
- joint RR_hip_joint: parent base_link -> torso
- joint imu_joint: parent base_link -> torso
- joint radar_joint: parent base_link -> torso

Commit message: Changes in workspace

File: go2_description/urdf/go2.xacro.urdf (robot description, URDF)
Before this commit: robot go2, 32 links, 31 joints
Links:
- removed link FL_calf
- removed link FL_calflower
- removed link FL_calflower1
- removed link FL_foot
- removed link FL_hip
- removed link FL_thigh
- removed link FR_calf
- removed link FR_calflower
- removed link FR_calflower1
- removed link FR_foot
- removed link FR_hip
- removed link FR_thigh
- removed link Head_lower
- removed link Head_upper
- removed link RL_calf
- removed link RL_calflower
- removed link RL_calflower1
- removed link RL_foot
- removed link RL_hip
- removed link RL_thigh
- removed link RR_calf
- removed link RR_calflower
- removed link RR_calflower1
- removed link RR_foot
- removed link RR_hip
- removed link RR_thigh
- removed link base_link
- removed link front_camera
- removed link imu
- removed link radar
- removed link torso
- removed link world
Joints:
- removed joint FL_calf_joint
- removed joint FL_calflower1_joint
- removed joint FL_calflower_joint
- removed joint FL_foot_joint
- removed joint FL_hip_joint
- removed joint FL_thigh_joint
- removed joint FR_calf_joint
- removed joint FR_calflower1_joint
- removed joint FR_calflower_joint
- removed joint FR_foot_joint
- removed joint FR_hip_joint
- removed joint FR_thigh_joint
- removed joint Head_lower_joint
- removed joint Head_upper_joint
- removed joint RL_calf_joint
- removed joint RL_calflower1_joint
- removed joint RL_calflower_joint
- removed joint RL_foot_joint
- removed joint RL_hip_joint
- removed joint RL_thigh_joint
- removed joint RR_calf_joint
- removed joint RR_calflower1_joint
- removed joint RR_calflower_joint
- removed joint RR_foot_joint
- removed joint RR_hip_joint
- removed joint RR_thigh_joint
- removed joint fixed
- removed joint front_camera_joint
- removed joint imu_joint
- removed joint joint_fixed_
- removed joint radar_joint
