Commit message: last modifications

File: go2_description/urdf/leg.xacro (robot description, xacro)
@@ -1,190 +1,159 @@
 <?xml version="1.0"?>
-<robot xmlns:xacro="http://ros.org/wiki/xacro">
-  <xacro:macro name="leg" params="name x y mirror_x mirror_y">
-    <!-- Set mesh variables -->
-    <xacro:property name="thigh_mesh" value="file://$(find go2_description)/dae/thigh.dae"/>
-    <xacro:property name="calf_mesh" value="file://$(find go2_description)/dae/calf.dae"/>
-    <xacro:property name="thigh_y" value="0.0955"/>
-    <xacro:if value="${mirror_y == -1}">
-      <xacro:property name="thigh_mesh" value="file://$(find go2_description)/dae/thigh_mirror.dae"/>
-      <xacro:property name="calf_mesh" value="file://$(find go2_description)/dae/calf_mirror.dae"/>
-      <xacro:property name="thigh_y" value="-0.0955"/>
-    </xacro:if>
-    <!-- Define properties values for the hip -->
-    <xacro:property name="com_x" value="${mirror_y * -0.0054}"/>
-    <xacro:property name="com_y" value="${mirror_x * 0.00194}"/>
-    <!-- <xacro:property name="vis_r" value="${(1 - mirror_x) * 3.1415/2}"/>
-    <xacro:property name="vis_p" value="${(1 - mirror_y) * 3.1415/2}"/>
-    <xacro:property name="vis_y" value="0"/> -->
-    <xacro:property name="ixx" value="0.00048"/>
-    <xacro:property name="iyy" value="0.000884"/>
-    <xacro:property name="izz" value="0.000596"/>
-    <xacro:property name="ixy" value="${mirror_x * -3.01e-6}"/>
-    <xacro:property name="ixz" value="${mirror_y * 1.11e-6}"/>
-    <xacro:property name="iyz" value="${mirror_x * mirror_y * 1.42e-6}"/>
-    <xacro:if value="${name == 'FL'}">
-      <xacro:property name="vis_r" value="0"/>
-      <xacro:property name="vis_p" value="0"/>
-      <xacro:property name="vis_y" value="0"/>
-    </xacro:if>
-    <xacro:if value="${name == 'FR'}">
-      <xacro:property name="vis_r" value="3.1415"/>
-      <xacro:property name="vis_p" value="0"/>
-      <xacro:property name="vis_y" value="0"/>
-    </xacro:if>
-    <xacro:if value="${name == 'RL'}">
-      <xacro:property name="vis_r" value="0"/>
-      <xacro:property name="vis_p" value="3.1415"/>
-      <xacro:property name="vis_y" value="0"/>
-    </xacro:if>
-    <xacro:if value="${name == 'RR'}">
-      <xacro:property name="vis_r" value="3.1415"/>
-      <xacro:property name="vis_p" value="3.1415"/>
-      <xacro:property name="vis_y" value="0"/>
-    </xacro:if>
-    <!-- Hip Link -->
-    <link name="${name}_hip">
-      <inertial>
-        <origin xyz="${com_x}  ${com_y} -0.000105" rpy="0 0 0"/>
-        <mass value="0.678"/>
-        <inertia ixx="${ixx}" ixy="${ixy}" ixz="${ixz}"
-                 iyy="${iyy}" iyz="${iyz}" izz="${izz}"/>
-      </inertial>
-      <visual>
-        <origin xyz="0 0 0" rpy="${vis_r} ${vis_p} ${vis_y}" />
-        <geometry>
-          <mesh filename="file://$(find go2_description)/dae/hip.dae"/>
-        </geometry>
-      </visual>
-      <collision>
-        <origin rpy="1.5707963267948966 0 0" xyz="0 ${mirror_y * 0.08} 0" />
-        <geometry>
-          <cylinder length="0.04" radius="0.046"/>
-        </geometry>
-      </collision>
-    </link>
-    <!-- Hip Joint -->
-    <joint name="${name}_hip_joint" type="revolute">
-      <origin xyz="${x} ${y} 0" rpy="0 0 0"/>
-      <parent link="base_link"/>
-      <child link="${name}_hip"/>
-      <axis xyz="1 0 0"/>
-      <limit lower="-1.0472" upper="1.0472" effort="23.7" velocity="30.1"/>
-    </joint>
-    <!-- Thigh Link -->
-    <link name="${name}_thigh">
-      <inertial>
-        <origin xyz="-0.00374 ${mirror_x * 0.0223} -0.0327" rpy="0 0 0"/>
-        <mass value="1.152"/>
-        <inertia ixx="0.00584" ixy="${mirror_x * -8.72e-5}" ixz="-0.000289"
-                 iyy="0.0058" iyz="${mirror_x * mirror_y * -0.000808}" izz="0.00103"/>
-      </inertial>
-      <visual>
-        <geometry>
-          <mesh filename="${thigh_mesh}"/>
-        </geometry>
-      </visual>
-      <collision>
-        <origin rpy="0 1.5707963267948966 0" xyz="0 0 -0.1065" />
-        <geometry>
-          <box size="0.213 0.0245 0.034"/>
-        </geometry>
-      </collision>
-    </link>
-    <!-- Thigh Joint -->
-    <joint name="${name}_thigh_joint" type="revolute">
-      <origin xyz="0 ${thigh_y} 0" rpy="0 0 0"/>
-      <parent link="${name}_hip"/>
-      <child link="${name}_thigh"/>
-      <axis xyz="0 1 0"/>
-      <limit lower="-1.5708" upper="3.4907" effort="23.7" velocity="30.1"/>
-    </joint>
-    <!-- Calf Link -->
-    <link name="${name}_calf">
-      <inertial>
-        <origin xyz="0.00548 ${mirror_x * 0.000975} -0.115" rpy="0 0 0" />
-        <mass value="0.154"/>
-        <inertia ixx="0.00108" ixy="${mirror_x * -3.40e-7}" ixz="0"
-                 iyy="0.0011" iyz="${mirror_x * mirror_y * -8.28e-6}" izz="3.29E-05"/>
-      </inertial>
-      <visual>
-        <geometry>
-          <mesh filename="${calf_mesh}"/>
-        </geometry>
-      </visual>
-      <collision>
-        <origin rpy="0 -0.2 0" xyz="0.008 0 -0.06" />
-        <geometry>
-          <cylinder length="0.12" radius="0.013"/>
-        </geometry>
-      </collision>
-    </link>
-    <!-- Calf Joint -->
-    <joint name="${name}_calf_joint" type="revolute">
-      <origin xyz="0 0 -0.213" rpy="0 0 0"/>
-      <parent link="${name}_thigh"/>
-      <child link="${name}_calf"/>
-      <axis xyz="0 1 0"/>
-      <limit lower="-2.7227" upper="-0.83776" effort="45.43" velocity="15.70"/>
-    </joint>
-    <!-- Calf lower Joint (only colision) -->
-    <link name="${name}_calflower">
-      <collision>
-        <origin rpy="0 0 0" xyz="0 0 0" />
-        <geometry>
-          <cylinder length="0.065" radius="0.011" />
-        </geometry>
-      </collision>
-    </link>
-    <!-- Calf lower Joint -->
-    <joint name="${name}_calflower_joint" type="fixed">
-      <origin xyz="0.020 0 -0.148" rpy="0 0.05 0" />
-      <parent link="${name}_calf" />
-      <child link="${name}_calflower" />
-      <axis xyz="0 1 0" />
-    </joint>
-    <!-- Calf lower 1 Joint (only colision) -->
-    <link name="${name}_calflower1">
-      <collision>
-        <origin rpy="0 0 0" xyz="0 0 0" />
-        <geometry>
-          <cylinder length="0.03" radius="0.0155" />
-        </geometry>
-      </collision>
-    </link>
-    <!-- Calf lower 1 Joint -->
-    <joint name="${name}_calflower1_joint" type="fixed">
-      <origin xyz="-0.01 0 -0.04" rpy="0 0.48 0" />
-      <parent link="${name}_calflower" />
-      <child link="${name}_calflower1" />
-      <axis xyz="0 0 0" />
-    </joint>
-    <!-- Foot Link -->
-    <link name="${name}_foot">
-      <inertial>
-        <origin xyz="0 0 0" rpy="0 0 0"/>
-        <mass value="0.04"/>
-        <inertia ixx="9.6e-06" ixy="0" ixz="0"
-                 iyy="9.6e-06" iyz="0" izz="9.6e-06"/>
-      </inertial>
-      <visual>
-        <origin xyz="0 0 0" rpy="0 0 0" />
-        <geometry>
-          <mesh filename="file://$(find go2_description)/dae/foot.dae"/>
-        </geometry>
-      </visual>
-      <collision>
-        <origin rpy="0 0 0" xyz="-0.002 0 0" />
-        <geometry>
-          <sphere radius="0.022"/>
-        </geometry>
-      </collision>
-    </link>
-    <!-- Foot Joint (Fixed) -->
-    <joint name="${name}_foot_joint" type="fixed" dont_collapse="true">
-      <origin xyz="0 0 -0.213" rpy="0 0 0"/>
-      <parent link="${name}_calf"/>
-      <child link="${name}_foot"/>
-    </joint>
-  </xacro:macro>
+<robot xmlns:xacro="http://www.ros.org/wiki/xacro">
+    <xacro:include filename="$(find go2_description)/urdf/transmission.xacro"/>
+    <xacro:macro name="leg" params="name mirror mirror_dae front_hind front_hind_dae">
+        <joint name="${name}_hip_joint" type="revolute">
+            <xacro:if value="${(mirror_dae == False) and (front_hind_dae == True)}">
+                <origin rpy="0 0 0" xyz="${leg_offset_x} ${-leg_offset_y} 0"/>
+            </xacro:if>
+            <xacro:if value="${(mirror_dae == True) and (front_hind_dae == True)}">
+                <origin rpy="0 0 0" xyz="${leg_offset_x} ${leg_offset_y} 0"/>
+            </xacro:if>
+            <xacro:if value="${(mirror_dae == False) and (front_hind_dae == False)}">
+                <origin rpy="0 0 0" xyz="${-leg_offset_x} ${-leg_offset_y} 0"/>
+            </xacro:if>
+            <xacro:if value="${(mirror_dae == True) and (front_hind_dae == False)}">
+                <origin rpy="0 0 0" xyz="${-leg_offset_x} ${leg_offset_y} 0"/>
+            </xacro:if>
+            <parent link="torso"/>
+            <child link="${name}_hip"/>
+            <axis xyz="1 0 0"/>
+            <dynamics damping="${damping}" friction="${friction}"/>
+            <xacro:if value="${(mirror_dae == True)}">
+                <limit effort="${hip_torque_max}" velocity="${hip_velocity_max}" lower="${hip_position_min}" upper="${hip_position_max}"/>
+            </xacro:if>
+            <xacro:if value="${(mirror_dae == False)}">
+                <limit effort="${hip_torque_max}" velocity="${hip_velocity_max}" lower="${-hip_position_max}" upper="${-hip_position_min}"/>
+            </xacro:if>
+        </joint>
+        <link name="${name}_hip">
+            <visual>
+                <xacro:if value="${(mirror_dae == True) and (front_hind_dae == True)}">
+                    <origin rpy="0 0 0" xyz="0 0 0"/>
+                </xacro:if>
+                <xacro:if value="${(mirror_dae == False) and (front_hind_dae == True)}">
+                    <origin rpy="${PI} 0 0" xyz="0 0 0"/>
+                </xacro:if>
+                <xacro:if value="${(mirror_dae == True) and (front_hind_dae == False)}">
+                    <origin rpy="0 ${PI} 0" xyz="0 0 0"/>
+                </xacro:if>
+                <xacro:if value="${(mirror_dae == False) and (front_hind_dae == False)}">
+                    <origin rpy="${PI} ${PI} 0" xyz="0 0 0"/>
+                </xacro:if>
+                <geometry>
+                    <mesh filename="file://$(find go2_description)/dae/hip.dae" scale="1 1 1"/>
+                </geometry>
+                <!-- <material name="orange"/> -->
+            </visual>
+            <collision>
+                <origin rpy="${PI/2.0} 0 0" xyz="0 ${hip_offset*mirror} 0"/>
+                <geometry>
+                    <cylinder length="${hip_length}" radius="${hip_radius}"/>
+                </geometry>
+            </collision>
+            <inertial>
+                <origin rpy="0 0 0" xyz="${hip_com_x*front_hind} ${hip_com_y*mirror} ${hip_com_z}"/>
+                <mass value="${hip_mass}"/>
+                <inertia
+                    ixx="${hip_ixx}" ixy="${hip_ixy*mirror*front_hind}" ixz="${hip_ixz*front_hind}"
+                    iyy="${hip_iyy}" iyz="${hip_iyz*mirror}"
+                    izz="${hip_izz}"/>
+            </inertial>
+        </link>
+        <joint name="${name}_thigh_joint" type="revolute">
+            <origin rpy="0 0 0" xyz="0 ${thigh_offset*mirror} 0"/>
+            <parent link="${name}_hip"/>
+            <child link="${name}_thigh"/>
+            <axis xyz="0 1 0"/>
+            <dynamics damping="${damping}" friction="${friction}"/>
+            <limit effort="${thigh_torque_max}" velocity="${thigh_velocity_max}" lower="${thigh_position_min}" upper="${thigh_position_max}"/>
+        </joint>
+        <link name="${name}_thigh">
+            <visual>
+                <origin rpy="0 0 0" xyz="0 0 0"/>
+                <geometry>
+                    <xacro:if value="${mirror_dae == True}">
+                        <mesh filename="file://$(find go2_description)/dae/thigh.dae" scale="1 1 1"/>
+                    </xacro:if>
+                    <xacro:if value="${mirror_dae == False}">
+                        <mesh filename="file://$(find go2_description)/dae/thigh_mirror.dae" scale="1 1 1"/>
+                    </xacro:if>
+                </geometry>
+                <!-- <material name="orange"/> -->
+            </visual>
+            <collision>
+                <origin rpy="0 ${PI/2.0} 0" xyz="0 0 ${-thigh_length/2.0}"/>
+                <geometry>
+                    <box size="${thigh_length} ${thigh_width} ${thigh_height}"/>
+                </geometry>
+            </collision>
+            <inertial>
+                <origin rpy="0 0 0" xyz="${thigh_com_x} ${thigh_com_y*mirror} ${thigh_com_z}"/>
+                <mass value="${thigh_mass}"/>
+                <inertia
+                    ixx="${thigh_ixx}" ixy="${thigh_ixy*mirror}" ixz="${thigh_ixz}"
+                    iyy="${thigh_iyy}" iyz="${thigh_iyz*mirror}"
+                    izz="${thigh_izz}"/>
+            </inertial>
+        </link>
+        <joint name="${name}_calf_joint" type="revolute">
+            <origin rpy="0 0 0" xyz="0 0 ${-thigh_length}"/>
+            <parent link="${name}_thigh"/>
+            <child link="${name}_calf"/>
+            <axis xyz="0 1 0"/>
+            <dynamics damping="${damping}" friction="${friction}"/>
+            <limit effort="${calf_torque_max}" velocity="${calf_velocity_max}" lower="${calf_position_min}" upper="${calf_position_max}"/>
+        </joint>
+        <link name="${name}_calf">
+            <visual>
+                <origin rpy="0 0 0" xyz="0 0 0"/>
+                <geometry>
+                    <mesh filename="file://$(find go2_description)/dae/calf.dae" scale="1 1 1"/>
+                </geometry>
+                <!-- <material name="orange"/> -->
+            </visual>
+            <collision>
+                <origin rpy="0 ${PI/2.0} 0" xyz="0 0 ${-calf_length/2.0}"/>
+                <geometry>
+                    <box size="${calf_length} ${calf_width} ${calf_height}"/>
+                </geometry>
+            </collision>
+            <inertial>
+                <origin rpy="0 0 0" xyz="${calf_com_x} ${calf_com_y} ${calf_com_z}"/>
+                <mass value="${calf_mass}"/>
+                <inertia
+                    ixx="${calf_ixx}" ixy="${calf_ixy}" ixz="${calf_ixz}"
+                    iyy="${calf_iyy}" iyz="${calf_iyz}"
+                    izz="${calf_izz}"/>
+            </inertial>
+        </link>
+        <joint name="${name}_foot_fixed" type="fixed">0
+            <origin rpy="0 0 0" xyz="0 0 ${-(calf_length)}"/>
+            <parent link="${name}_calf"/>
+            <child link="${name}_foot"/>
+        </joint>
+        <link name="${name}_foot">
+            <visual>
+                <origin rpy="0 0 0" xyz="0 0 0"/>
+                <geometry>
+                    <sphere radius="${foot_radius-0.01}"/>
+                </geometry>
+                <!-- <material name="orange"/> -->
+            </visual>
+            <collision>
+                <origin rpy="0 0 0" xyz="0 0 0"/>
+                <geometry>
+                    <sphere radius="${foot_radius}"/>
+                </geometry>
+            </collision>
+            <inertial>
+                <mass value="${foot_mass}"/>
+                <inertia
+                    ixx="${(2*foot_mass)/5.0*(foot_radius*foot_radius)}" ixy="0.0" ixz="0.0"
+                    iyy="${(2*foot_mass)/5.0*(foot_radius*foot_radius)}" iyz="0.0"
+                    izz="${(2*foot_mass)/5.0*(foot_radius*foot_radius)}"/>
+            </inertial>
+        </link>
+        <!-- <xacro:leg_transmission name="${name}"/> -->
+    </xacro:macro>
 </robot>

File: go2_description/urdf/sensors.xacro (robot description, xacro)
@@ -38,5 +38,5 @@
     </link>
     <joint name="imu_joint" type="fixed">
-      <parent link="base_link"/>
+      <parent link="torso"/>
       <child link="imu"/>
       <origin xyz="-0.02557 0 0.04232" rpy="0 0 0"/>
@@ -44,5 +44,5 @@
     </joint>
     <!-- ====================== FRONT LIDAR CAMERA ====================== -->
-    <link name="radar">
+    <!-- <link name="radar">
       <inertial>
         <origin xyz="0 0 0" rpy="0 0 0"/>
@@ -57,5 +57,5 @@
       <origin xyz="0.28945 0 -0.046825" rpy="0 2.8782 0"/>
       <axis xyz="0 0 0"/>
-    </joint>
+    </joint> -->
   </xacro:macro>
 </robot>

File: go2_description/urdf/torso.xacro (robot description, xacro)
@@ -2,54 +2,47 @@
 <robot xmlns:xacro="http://ros.org/wiki/xacro">
     <xacro:macro name="torso" params="simulation fixed_base">
+    <link name="world" />
+      <joint name="fixed" type="fixed">
+        <parent link="world"/>
+        <child link="base"/>
+        <origin xyz="0 0 1"/>
+      </joint>
     <!-- World frame -->
-    <link name="world"/>
-    <!-- <xacro:if value="${simulation}">
-      <xacro:if value="${fixed_base}">
-        <joint name="world_to_base" type="fixed">
-          <parent link="world"/>
-          <child link="base_link"/>
-          <origin xyz="0 0 1"/>
+        <link name="base">
+            <visual>
+                <origin rpy="0 0 0" xyz="0 0 0"/>
+                <geometry>
+                    <box size="0.001 0.001 0.001"/>
+                </geometry>
+            </visual>
+        </link>
+        <joint name="floating_base" type="fixed">
+            <origin rpy="0 0 0" xyz="0 0 0"/>
+            <parent link="base"/>
+            <child link="torso"/>
         </joint>
-      </xacro:if>
-    </xacro:if> -->
-    <!-- Movable base in simulation OR real robot -->
-    <!-- <xacro:unless value="${fixed_base}"> -->
-      <link name="odom"/>
-      <joint name="world_to_odom" type="fixed">
-        <parent link="world"/>
-        <child link="odom"/>
-      </joint>
-      <joint name="odom_to_base" type="fixed">
-        <parent link="odom"/>
-        <child link="base_link"/>
-      </joint>
-    <!-- </xacro:unless> -->
-    <!-- Base link -->
-    <link name="base_link">
-      <inertial>
-        <origin xyz="0.021112 0 -0.005366" rpy="0 0 0"/>
-        <mass value="6.921"/>
-        <inertia ixx="0.02448" ixy="0.00012166" ixz="0.0014849"
-                 iyy="0.098077" iyz="-3.12E-05" izz="0.107"/>
-      </inertial>
-      <visual>
-        <origin xyz="0 0 0" rpy="0 0 0"/>
-        <geometry>
-          <mesh filename="file://$(find go2_description)/dae/base.dae"/>
-        </geometry>
-      </visual>
-      <collision>
-        <origin xyz="0 0 0" rpy="0 0 0"/>
-        <geometry>
-          <box size="0.3762 0.0935 0.114"/>
-        </geometry>
-      </collision>
+        <link name="torso">
+            <visual>
+                <origin rpy="0 0 0" xyz="0 0 0"/>
+                <geometry>
+                    <mesh filename="file://$(find go2_description)/dae/base.dae"/>
+                </geometry>
+                <!-- <material name="orange"/> -->
+            </visual>
+            <collision>
+                <origin rpy="0 0 0" xyz="0 0 0"/>
+                <geometry>
+                    <box size="${trunk_length} ${trunk_width} ${trunk_height}"/>
+                </geometry>
+            </collision>
+            <inertial>
+                <origin rpy="0 0 0" xyz="${trunk_com_x} ${trunk_com_y} ${trunk_com_z}"/>
+                <mass value="${trunk_mass}"/>
+                <inertia
+                    ixx="${trunk_ixx}" ixy="${trunk_ixy}" ixz="${trunk_ixz}"
+                    iyy="${trunk_iyy}" iyz="${trunk_iyz}"
+                    izz="${trunk_izz}"/>
+            </inertial>
     </link>
-    <joint name="base_footprint_joint" type="fixed">
-      <parent link="base_link"/>
-      <child link="base_footprint"/>
-      <origin xyz="0 0 0" rpy="0 0 0"/>
-    </joint>
-    <link name="base_footprint"/>
     <!-- ====================== HEAD UPPER ====================== -->
     <link name="Head_upper">
@@ -68,5 +61,5 @@
     </link>
     <joint name="Head_upper_joint" type="fixed" dont_collapse="true">
-      <parent link="base_link"/>
+      <parent link="torso"/>
       <child link="Head_upper"/>
       <origin xyz="0.285 0 0.01" rpy="0 0 0"/>
