Commit message: minnor changes

File: go2_description/urdf/sensors.xacro (robot description, xacro)
@@ -44,5 +44,5 @@
     </joint>
     <!-- ====================== FRONT LIDAR CAMERA ====================== -->
-    <!-- <link name="radar">
+        <link name="radar">
       <inertial>
         <origin xyz="0 0 0" rpy="0 0 0"/>
@@ -57,5 +57,11 @@
       <origin xyz="0.28945 0 -0.046825" rpy="0 2.8782 0"/>
       <axis xyz="0 0 0"/>
-    </joint> -->
+    </joint>
+    <link name="utlidar_lidar"/>
+    <joint name="utlidar_lidar_joint" type="fixed">
+      <parent link="radar"/>
+      <child link="utlidar_lidar"/>
+      <origin xyz="0 0 0" rpy="0 0 0"/>
+    </joint>
   </xacro:macro>
 </robot>
